File: hardware/v0.3/PiHAT_v0.3.brd (EAGLE design)
At the start: 65 x 56.5 mm, 39 parts, among them IC1 BMP280, J1 FTDI, J3 ISP, U1 ATMEGA328P, U2 TSL2561, U3 OPA344, U6 ADMP401, U7 SHT31/35, U8 CCS811, Y1 16MHZ

Commit message: BOM adjustments
Parts:
- removed C1, C6: 0.1uF, SparkFun-Passives:0805
- added C11, C7: 0.1uF, SparkFun-Passives:0805
Connections:
- net GND: now also C11.2, C7.2; no longer C1.2, C6.1
- net VCC: now also C11.1, C7.1; no longer C1.1, C6.2
Routing:
- net SCL: track 98.2 -> 96.3 mm
Changed lines of the file:
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@@
 <?xml version="1.0" encoding="utf-8"?>
 <!DOCTYPE eagle SYSTEM "eagle.dtd">
-<eagle version="7.7.0">
+<eagle version="7.6.0">
 <drawing>
 <settings>
@@
 <attribute name="DIGIKEY#" value="311-1088-1-ND" x="26.9494" y="6.096" size="1.778" layer="27" display="off"/>
 <attribute name="MPN" value="CC0603KRX7R7BB104" x="26.9494" y="6.096" size="1.778" layer="27" display="off"/>
-<attribute name="MOUSER#" value="603-RC0805FR-07100RL" x="26.9494" y="6.096" size="1.778" layer="27" display="off"/>
+<attribute name="MOUSER#" value="603-CC603KRX7R7BB104" x="26.9494" y="6.096" size="1.778" layer="27" display="off"/>
 </element>
 <element name="C4" library="SparkFun-Passives" package="0805" value="0.1uF" x="10.795" y="2.921" smashed="yes" rot="R270">
@@
 <attribute name="VALUE" x="39.6048" y="0.9404" size="0.8128" layer="21" font="vector" rot="R180"/>
 </element>
-<element name="C1" library="SparkFun-Passives" package="0805" value="0.1uF" x="34.29" y="5.0292" smashed="yes" rot="R90">
-<attribute name="VALUE" x="33.0454" y="3.7084" size="0.8128" layer="21" font="vector" rot="R90"/>
-</element>
-<element name="C6" library="SparkFun-Passives" package="0805" value="0.1uF" x="37.3888" y="6.096" smashed="yes" rot="R180">
-<attribute name="VALUE" x="39.3192" y="8.0518" size="0.8128" layer="21" font="vector" rot="R180"/>
-</element>
 <element name="JP1" library="SparkFun-Passives" package="PAD-JUMPER-2-NC_BY_PASTE_YES_SILK_FULL_BOX" value="SDA" x="59.5884" y="45.466" smashed="yes" rot="MR90">
 <attribute name="VALUE" x="61.7474" y="46.619" size="0.8128" layer="22" font="vector" rot="MR270"/>
@@
 <element name="JP2" library="SparkFun-Passives" package="PAD-JUMPER-2-NC_BY_PASTE_YES_SILK_FULL_BOX" value="SCL" x="56.9976" y="45.466" smashed="yes" rot="MR90">
 <attribute name="VALUE" x="55.6006" y="46.4666" size="0.8128" layer="22" font="vector" rot="SMR270"/>
+</element>
+<element name="C7" library="SparkFun-Passives" package="0805" value="0.1uF" x="37.3888" y="6.1976">
+<attribute name="DIGIKEY#" value="311-1088-1-ND" x="37.3888" y="6.1976" size="1.778" layer="27" display="off"/>
+<attribute name="MOUSER#" value="603-CC603KRX7R7BB104" x="37.3888" y="6.1976" size="1.778" layer="27" display="off"/>
+<attribute name="MPN" value="CC0603KRX7R7BB104" x="37.3888" y="6.1976" size="1.778" layer="27" display="off"/>
+</element>
+<element name="C11" library="SparkFun-Passives" package="0805" value="0.1uF" x="33.8836" y="5.0292" rot="R90">
+<attribute name="DIGIKEY#" value="311-1088-1-ND" x="33.8836" y="5.0292" size="1.778" layer="27" rot="R90" display="off"/>
+<attribute name="MOUSER#" value="603-CC603KRX7R7BB104" x="33.8836" y="5.0292" size="1.778" layer="27" rot="R90" display="off"/>
+<attribute name="MPN" value="CC0603KRX7R7BB104" x="33.8836" y="5.0292" size="1.778" layer="27" rot="R90" display="off"/>
 </element>
 </elements>
@@
 <via x="28.702" y="1.6256" extent="1-16" drill="0.381" diameter="0.254"/>
 <wire x1="28.702" y1="1.6256" x2="28.702" y2="0.6604" width="0.254" layer="16"/>
-<wire x1="28.702" y1="1.6256" x2="34.544" y2="1.6256" width="0.254" layer="16"/>
-<via x="39.3192" y="1.4224" extent="1-16" drill="0.381" diameter="0.254"/>
+<via x="39.3192" y="1.6256" extent="1-16" drill="0.381" diameter="0.254"/>
 <wire x1="38.097" y1="2.1844" x2="38.0872" y2="2.1746" width="0.254" layer="1"/>
 <wire x1="17.3228" y1="1.016" x2="18.4912" y2="-0.1524" width="0.254" layer="16" curve="90"/>
 <wire x1="27.8892" y1="-0.1524" x2="28.702" y2="0.6604" width="0.254" layer="16" curve="90"/>
-<wire x1="34.544" y1="1.6256" x2="35.306" y2="0.8636" width="0.254" layer="16" curve="-90"/>
-<wire x1="35.306" y1="0.8636" x2="35.306" y2="0.7112" width="0.254" layer="16"/>
-<wire x1="35.306" y1="0.7112" x2="36.068" y2="-0.0508" width="0.254" layer="16" curve="90"/>
-<wire x1="39.3192" y1="0.762" x2="38.5064" y2="-0.0508" width="0.254" layer="16" curve="-90"/>
-<wire x1="38.5064" y1="-0.0508" x2="36.068" y2="-0.0508" width="0.254" layer="16"/>
-<wire x1="38.097" y1="2.1844" x2="38.5572" y2="2.1844" width="0.254" layer="1"/>
-<wire x1="38.5572" y1="2.1844" x2="39.3192" y2="1.4224" width="0.254" layer="1" curve="-90"/>
-<wire x1="39.3192" y1="0.762" x2="39.3192" y2="1.4224" width="0.254" layer="16"/>
+<wire x1="38.097" y1="2.1844" x2="38.7604" y2="2.1844" width="0.254" layer="1"/>
 <wire x1="28.0566" y1="2.271" x2="28.702" y2="1.6256" width="0.254" layer="1" curve="-90"/>
 <wire x1="45.9486" y1="31.35" x2="47.1124" y2="31.35" width="0.254" layer="1"/>
@@
 <wire x1="43.5864" y1="31.3436" x2="45.9422" y2="31.3436" width="0.254" layer="1"/>
 <wire x1="45.9422" y1="31.3436" x2="45.9486" y2="31.35" width="0.254" layer="1" curve="90"/>
-<wire x1="39.3192" y1="1.4224" x2="39.5732" y2="1.4224" width="0.254" layer="16"/>
-<wire x1="39.5732" y1="1.4224" x2="41.0464" y2="2.8956" width="0.254" layer="16" curve="90"/>
 <wire x1="41.0464" y1="2.8956" x2="41.0464" y2="28.8036" width="0.254" layer="16"/>
 <wire x1="58.9792" y1="38.4172" x2="57.01" y2="38.4172" width="0.254" layer="1"/>
@@
 <contactref element="JP2" pad="1"/>
 <wire x1="56.9976" y1="38.4048" x2="56.9976" y2="45.0541" width="0.254" layer="16"/>
+<wire x1="28.702" y1="1.6256" x2="39.3192" y2="1.6256" width="0.254" layer="16"/>
+<wire x1="38.7604" y1="2.1844" x2="39.3192" y2="1.6256" width="0.254" layer="1" curve="-90"/>
+<wire x1="41.0464" y1="2.8956" x2="39.7764" y2="1.6256" width="0.254" layer="16" curve="-90"/>
+<wire x1="39.7764" y1="1.6256" x2="39.3192" y2="1.6256" width="0.254" layer="16"/>
 </signal>
 <signal name="GPIO4">
@@
 <contactref element="IC1" pad="7"/>
 <contactref element="IC1" pad="1"/>
-<contactref element="C6" pad="1"/>
-<contactref element="C1" pad="2"/>
 <wire x1="15.399" y1="2.798" x2="14.474" y2="2.798" width="0.254" layer="1"/>
 <wire x1="14.474" y1="2.798" x2="14.224" y2="3.048" width="0.254" layer="1"/>
+<contactref element="C7" pad="2"/>
+<contactref element="C11" pad="2"/>
 <wire x1="41.256" y1="36.0426" x2="42.856" y2="36.0426" width="0" layer="19" extent="1-1"/>
 </signal>
@@
 <contactref element="J1" pad="VCC"/>
 <contactref element="IC1" pad="8"/>
-<contactref element="C6" pad="2"/>
 <contactref element="IC1" pad="6"/>
 <contactref element="IC1" pad="5"/>
-<contactref element="C1" pad="1"/>
 <wire x1="10.8966" y1="12.689" x2="9.7934" y2="12.689" width="0.4064" layer="1"/>
 <wire x1="9.144" y1="12.0396" x2="9.144" y2="4.2672" width="0.4064" layer="1"/>
@@
 <wire x1="39.1668" y1="25.2984" x2="39.656" y2="25.7876" width="0.4064" layer="1" curve="90"/>
 <wire x1="36.4888" y1="25.2332" x2="36.4236" y2="25.2984" width="0.254" layer="1"/>
-<wire x1="36.4872" y1="4.1246" x2="34.2946" y2="4.1246" width="0.254" layer="1"/>
-<wire x1="34.2946" y1="4.1246" x2="34.29" y2="4.1292" width="0.254" layer="1"/>
-<wire x1="36.4872" y1="4.1246" x2="36.4872" y2="6.0944" width="0.4064" layer="1"/>
-<wire x1="36.4872" y1="6.0944" x2="36.4888" y2="6.096" width="0.254" layer="1"/>
 <wire x1="36.4872" y1="2.8246" x2="36.4872" y2="2.1746" width="0.254" layer="1"/>
-<wire x1="36.4872" y1="2.8246" x2="35.5946" y2="2.8246" width="0.254" layer="1"/>
-<wire x1="35.5946" y1="2.8246" x2="34.29" y2="4.1292" width="0.254" layer="1" curve="-90"/>
 <wire x1="9.6012" y1="3.81" x2="9.144" y2="4.2672" width="0.4064" layer="1" curve="-90"/>
 <wire x1="9.144" y1="12.0396" x2="9.7934" y2="12.689" width="0.4064" layer="1" curve="-90"/>
@@
 <wire x1="7.62" y1="28.0924" x2="8.9408" y2="28.0924" width="0.4064" layer="1"/>
 <wire x1="8.9408" y1="28.0924" x2="10.4648" y2="29.6164" width="0.4064" layer="1" curve="90"/>
-<wire x1="10.4648" y1="29.6164" x2="10.4648" y2="30.2768" width="0.4064" layer="1"/>
-<wire x1="10.4648" y1="30.2768" x2="12.446" y2="32.258" width="0.4064" layer="1" curve="-90"/>
-<wire x1="12.446" y1="32.258" x2="14.5288" y2="32.258" width="0.4064" layer="1"/>
-<wire x1="14.5288" y1="32.258" x2="16.4592" y2="30.3276" width="0.4064" layer="1" curve="-90"/>
 <wire x1="16.4592" y1="30.3276" x2="16.4592" y2="29.1592" width="0.4064" layer="1"/>
 <wire x1="16.4592" y1="29.1592" x2="24.384" y2="29.1592" width="0.4064" layer="1"/>
@@
 <wire x1="26.0604" y1="27.4828" x2="26.0604" y2="22.5552" width="0.4064" layer="1"/>
 <wire x1="26.0604" y1="22.5552" x2="26.0494" y2="22.5442" width="0.254" layer="1" curve="-90"/>
-<wire x1="36.4888" y1="6.096" x2="36.4888" y2="22.6712" width="0.4064" layer="1"/>
-<wire x1="36.4888" y1="22.6712" x2="39.116" y2="25.2984" width="0.4064" layer="1" curve="-90"/>
 <wire x1="12.4096" y1="11.176" x2="24.0174" y2="11.176" width="0.4064" layer="1"/>
 <wire x1="24.0174" y1="11.176" x2="26.0494" y2="13.208" width="0.4064" layer="1" curve="90"/>
@@
 <wire x1="42.056" y1="36.0426" x2="42.056" y2="38.2316" width="0.4064" layer="1"/>
 <wire x1="42.056" y1="38.2316" x2="42.7626" y2="38.9382" width="0.4064" layer="1" curve="-90"/>
+<wire x1="10.4648" y1="29.6164" x2="10.4648" y2="30.1752" width="0.4064" layer="1"/>
+<wire x1="10.4648" y1="30.1752" x2="12.0904" y2="31.8008" width="0.4064" layer="1" curve="-90"/>
+<wire x1="12.0904" y1="31.8008" x2="14.986" y2="31.8008" width="0.4064" layer="1"/>
+<wire x1="14.986" y1="31.8008" x2="16.4592" y2="30.3276" width="0.4064" layer="1" curve="-90"/>
+<contactref element="C7" pad="1"/>
+<contactref element="C11" pad="1"/>
+<wire x1="36.4888" y1="6.1976" x2="36.4888" y2="4.1262" width="0.254" layer="1"/>
+<wire x1="36.4888" y1="4.1262" x2="36.4872" y2="4.1246" width="0.254" layer="1" curve="-90"/>
+<wire x1="39.116" y1="25.2984" x2="36.4888" y2="22.6712" width="0.4064" layer="1" curve="90"/>
+<wire x1="36.4888" y1="22.6712" x2="36.4888" y2="6.1976" width="0.4064" layer="1"/>
+<wire x1="33.8836" y1="4.1292" x2="33.8882" y2="4.1246" width="0.254" layer="1" curve="90"/>
+<wire x1="33.8882" y1="4.1246" x2="36.4872" y2="4.1246" width="0.254" layer="1"/>
+<wire x1="36.4872" y1="2.8246" x2="35.1882" y2="2.8246" width="0.254" layer="1"/>
+<wire x1="35.1882" y1="2.8246" x2="33.8836" y2="4.1292" width="0.254" layer="1" curve="-90"/>
 </signal>
 <signal name="D5">

Commit message: Updated all attributes for BOM
Fixed digikey and mouser numbers
Changed lines of the file:
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@@
 </element>
 <element name="C3" library="SparkFun-Passives" package="0805" value="0.1uF" x="26.9494" y="6.096" smashed="yes">
-<attribute name="VALUE" x="25.4762" y="7.4676" size="0.8128" layer="21" font="vector"/>
+<attribute name="VALUE" x="25.6286" y="7.4168" size="0.8128" layer="21" font="vector"/>
 <attribute name="DIGIKEY#" value="311-1088-1-ND" x="26.9494" y="6.096" size="1.778" layer="27" display="off"/>
 <attribute name="MPN" value="CC0603KRX7R7BB104" x="26.9494" y="6.096" size="1.778" layer="27" display="off"/>
@@
 <element name="R8" library="SparkFun-Passives" package="0805" value="100K" x="62.4586" y="11.2014" smashed="yes" rot="R180">
 <attribute name="VALUE" x="63.9826" y="13.1064" size="0.8128" layer="21" font="vector" rot="R180"/>
-<attribute name="DIGIKEY#" value="541-82.0CCT-ND" x="62.4586" y="11.2014" size="1.778" layer="27" rot="R180" display="off"/>
+<attribute name="DIGIKEY#" value="311-100KCRCT-ND" x="62.4586" y="11.2014" size="1.778" layer="27" rot="R180" display="off"/>
 <attribute name="MPN" value="RC0805FR-07100KL" x="62.4586" y="11.2014" size="1.778" layer="27" rot="R180" display="off"/>
 <attribute name="MOUSER#" value="603-RC0805FR-07100KL" x="62.4586" y="11.2014" size="1.778" layer="27" rot="R180" display="off"/>
@@
 </element>
 <element name="R9" library="SparkFun-Passives" package="0805" value="100K" x="59.8932" y="33.5788" smashed="yes" rot="R180">
-<attribute name="DIGIKEY#" value="541-82.0CCT-ND" x="59.8932" y="33.5788" size="1.778" layer="27" rot="R180" display="off"/>
+<attribute name="DIGIKEY#" value="311-100KCRCT-ND" x="59.8932" y="33.5788" size="1.778" layer="27" rot="R180" display="off"/>
 <attribute name="VALUE" x="58.1152" y="34.0106" size="0.8128" layer="21" font="vector" rot="R180"/>
 <attribute name="MPN" value="RC0805FR-07100KL" x="59.8932" y="33.5788" size="1.778" layer="27" rot="R180" display="off"/>
@@
 <element name="J1" library="SparkFun-Connectors" package="FTDI_BASIC" value="FTDI" x="7.62" y="20.4724" smashed="yes" rot="R90">
 <attribute name="VALUE" x="8.7884" y="35.687" size="0.6096" layer="21" font="vector" rot="R180"/>
-<attribute name="MPN" value="FT231XS-R" x="7.62" y="20.4724" size="1.778" layer="27" rot="R90" display="off"/>
-<attribute name="DIGIKEY#" value="768-1129-1-ND" x="7.62" y="20.4724" size="1.778" layer="27" rot="R90" display="off"/>
-<attribute name="MOUSER#" value="895-FT231XS-R" x="7.62" y="20.4724" size="1.778" layer="27" rot="R90" display="off"/>
+<attribute name="NO_BOM" value="TRUE" x="7.62" y="20.4724" size="1.778" layer="27" rot="R90" display="off"/>
 </element>
 <element name="J3" library="SparkFun-Connectors" package="2X3" value="ISP" x="13.9192" y="29.1592" smashed="yes" rot="R270">
@@
 <element name="IC1" library="bosch-bmp280" package="BMP280" value="BMP280" x="37.2872" y="3.1496" smashed="yes" rot="R90">
 <attribute name="VALUE" x="39.6048" y="0.9404" size="0.8128" layer="21" font="vector" rot="R180"/>
+<attribute name="DIGIKEY#" value="828-1064-1-ND" x="37.2872" y="3.1496" size="1.778" layer="27" rot="R90" display="off"/>
+<attribute name="MANF" value="BMP280" x="37.2872" y="3.1496" size="1.778" layer="27" rot="R90" display="off"/>
+<attribute name="MOUSER#" value="262-BMP280" x="37.2872" y="3.1496" size="1.778" layer="27" rot="R90" display="off"/>
 </element>
 <element name="JP1" library="SparkFun-Passives" package="PAD-JUMPER-2-NC_BY_PASTE_YES_SILK_FULL_BOX" value="SDA" x="59.5884" y="45.466" smashed="yes" rot="MR90">
@@
 <attribute name="VALUE" x="55.6006" y="46.4666" size="0.8128" layer="22" font="vector" rot="SMR270"/>
 </element>
-<element name="C7" library="SparkFun-Passives" package="0805" value="0.1uF" x="37.3888" y="6.1976">
+<element name="C7" library="SparkFun-Passives" package="0805" value="0.1uF" x="37.3888" y="6.1976" smashed="yes">
 <attribute name="DIGIKEY#" value="311-1088-1-ND" x="37.3888" y="6.1976" size="1.778" layer="27" display="off"/>
 <attribute name="MOUSER#" value="603-CC603KRX7R7BB104" x="37.3888" y="6.1976" size="1.778" layer="27" display="off"/>
 <attribute name="MPN" value="CC0603KRX7R7BB104" x="37.3888" y="6.1976" size="1.778" layer="27" display="off"/>
+<attribute name="VALUE" x="35.9664" y="7.4422" size="0.8128" layer="21" font="vector"/>
 </element>
-<element name="C11" library="SparkFun-Passives" package="0805" value="0.1uF" x="33.8836" y="5.0292" rot="R90">
+<element name="C11" library="SparkFun-Passives" package="0805" value="0.1uF" x="33.8836" y="5.0292" smashed="yes" rot="R90">
 <attribute name="DIGIKEY#" value="311-1088-1-ND" x="33.8836" y="5.0292" size="1.778" layer="27" rot="R90" display="off"/>
 <attribute name="MOUSER#" value="603-CC603KRX7R7BB104" x="33.8836" y="5.0292" size="1.778" layer="27" rot="R90" display="off"/>
 <attribute name="MPN" value="CC0603KRX7R7BB104" x="33.8836" y="5.0292" size="1.778" layer="27" rot="R90" display="off"/>
+<attribute name="VALUE" x="32.4866" y="3.7592" size="0.8128" layer="21" font="vector" rot="R90"/>
 </element>
 </elements>
