File: hardware/v0.3/PiHAT_v0.3.sch (EAGLE design)
At the start: 39 parts, among them IC1 BMP280, J1 FTDI, J3 ISP, U1 ATMEGA328P, U2 TSL2561, U3 OPA344, U6 ADMP401, U7 SHT31/35, U8 CCS811, Y1 16MHZ

Commit message: Updated LED attributes
Changed MPN from 0603 to 0805 part
Parts:
- LED1, LED2, LED3: DIGIKEY# 475-1196-1-ND -> (none); MOUSER# 720-LYL29KH1K226Z -> (none); MPN LY L29K-H1K2-26-Z -> LTST-C170TBKT
Changed lines of the file:
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@@
 <part name="SUPPLY7" library="SparkFun-Aesthetics" deviceset="VCC" device=""/>
 <part name="LED1" library="adafruit" deviceset="LED" device="CHIPLED_0805">
-<attribute name="DIGIKEY#" value="475-1196-1-ND"/>
-<attribute name="MOUSER#" value="720-LYL29KH1K226Z"/>
-<attribute name="MPN" value="LY L29K-H1K2-26-Z"/>
+<attribute name="MPN" value="LTST-C170TBKT"/>
 </part>
 <part name="GND8" library="SparkFun-Aesthetics" deviceset="GND" device=""/>
@@
 <part name="LED3" library="adafruit" deviceset="LED" device="CHIPLED_0805">
 <attribute name="DESCRIPTION" value="LED"/>
-<attribute name="DIGIKEY#" value="475-1196-1-ND"/>
-<attribute name="MOUSER#" value="720-LYL29KH1K226Z"/>
-<attribute name="MPN" value="LY L29K-H1K2-26-Z"/>
+<attribute name="MPN" value="LTST-C170TBKT"/>
 </part>
 <part name="R2" library="SparkFun-Resistors" deviceset="RESISTOR" device="0805-RES" value="47">
@@
 <part name="LED2" library="adafruit" deviceset="LED" device="CHIPLED_0805">
 <attribute name="DESCRIPTION" value="LED"/>
-<attribute name="DIGIKEY#" value="475-1196-1-ND"/>
-<attribute name="MOUSER#" value="720-LYL29KH1K226Z"/>
-<attribute name="MPN" value="LY L29K-H1K2-26-Z"/>
+<attribute name="MPN" value="LTST-C170TBKT"/>
 </part>
 <part name="J1" library="SparkFun-Connectors" deviceset="FTDI_BASIC" device="PTH" value="FTDI">
@@
 <instance part="LED1" gate="G$1" x="513.08" y="60.96" rot="R90">
 <attribute name="MPN" x="513.08" y="60.96" size="1.778" layer="96" rot="R270" display="off"/>
-<attribute name="DIGIKEY#" x="513.08" y="60.96" size="1.778" layer="96" rot="R90" display="off"/>
-<attribute name="MOUSER#" x="513.08" y="60.96" size="1.778" layer="96" rot="R90" display="off"/>
 </instance>
 <instance part="GND8" gate="1" x="520.7" y="50.8"/>
@@
 <instance part="LED3" gate="G$1" x="170.18" y="78.74" rot="R270">
 <attribute name="MPN" x="170.18" y="78.74" size="1.778" layer="96" rot="R90" display="off"/>
-<attribute name="DIGIKEY#" x="170.18" y="78.74" size="1.778" layer="96" rot="R270" display="off"/>
 <attribute name="DESCRIPTION" x="170.18" y="78.74" size="1.778" layer="96" rot="R270" display="off"/>
-<attribute name="MOUSER#" x="170.18" y="78.74" size="1.778" layer="96" rot="R270" display="off"/>
 </instance>
 <instance part="R2" gate="G$1" x="182.88" y="78.74">
@@
 <instance part="LED2" gate="G$1" x="170.18" y="88.9" rot="R270">
 <attribute name="MPN" x="170.18" y="88.9" size="1.778" layer="96" rot="R90" display="off"/>
-<attribute name="DIGIKEY#" x="170.18" y="88.9" size="1.778" layer="96" rot="R270" display="off"/>
 <attribute name="DESCRIPTION" x="170.18" y="88.9" size="1.778" layer="96" rot="R270" display="off"/>
-<attribute name="MOUSER#" x="170.18" y="88.9" size="1.778" layer="96" rot="R270" display="off"/>
 </instance>
 <instance part="J1" gate="G$1" x="200.66" y="-78.74">

Commit message: Removed Digikey and Mouser numbers to avoid confusion
Parts:
- C10, C11, C12, C15, C3, C4, C5, C7: DIGIKEY# 311-1088-1-ND -> (none); MOUSER# 603-CC603KRX7R7BB104 -> (none)
- C2: DIGIKEY# 311-1111-1-ND -> (none); MOUSER# 603-CC805JRNPO9BN101 -> (none)
- C8: DIGIKEY# 311-1871-1-ND -> (none); MOUSER# 603-CC805KKX5R8BB475 -> (none)
- C9: DIGIKEY# 311-1365-1-ND -> (none); MOUSER# 603-CC805KKX7R7BB105 -> (none)
- IC1: DIGIKEY# 828-1064-1-ND -> (none); MANF BMP280 -> (none); MOUSER# 262-BMP280 -> (none); MPN (none) -> BMP280
- JP1, JP2: NO_BOM (none) -> TRUE
- LED2, LED3: DESCRIPTION LED -> (none)
- R1, R13, R5, R6, R7: DIGIKEY# 311-10KARCT-ND -> (none); MOUSER# 603-RC0805JR-0710KL -> (none)
- R10, R2, R4: DIGIKEY# 311-47ARCT-ND -> (none); MOUSER# 603-RC0805JR-0747RL -> (none)
- R3: DIGIKEY# YAG1814CT-ND -> (none); MOUSER# 603-RT0805BRD071K5L -> (none)
- R8, R9: DIGIKEY# 311-100KCRCT-ND -> (none); MOUSER# 603-RC0805FR-07100KL -> (none)
- RESET: DIGIKEY# CKN9104CT-ND -> (none); MOUSER# 611-PTS525SM15SMTR2 -> (none)
- U1: DIGIKEY# ATMEGA328P-AU-ND -> (none); MOUSER# 556-ATMEGA328P-AU -> (none)
- U2: DIGIKEY# TSL2561-FNCT-ND -> (none); MANF AMS-TAOS-USA-Inc. -> (none); MOUSER# 856-TSL2561T -> (none)
- U3: DIGIKEY# 296-41475-1-ND -> (none); MOUSER# 595-OPA344NA/3K -> (none)
- U6: DIGIKEY# INMP401ACEZ-R7CT-ND -> (none)
- U7: DIGIKEY# 1649-1011-1-ND -> (none); MOUSER# 403-SHT31-DIS-B -> (none)
- U8: MANF AMS -> (none)
- Y1: DIGIKEY# 490-1198-1-ND -> (none); MOUSER# 81-CSTCE16M0V53-R0 -> (none)
